File: hardware/contapassi.kicad_pcb (KiCad board)
At the start: 4 copper layers, 24 x 41 mm, 35 parts, among them J1 piazzole pogo, J2 cella LiPo, Q1 AO3401A, U1 E73-2G4M08S1C, U2 LSM6DSV16XTR, U3 W25Q256JVEIQ, U4 MCP73831T-2ATI/OT, Y1 32.768kHz

Commit message: Add routing functionality for PCB generation
- Introduced a new routing module (`route.py`) to handle the routing of pads on the PCB.
- Implemented a grid-based routing algorithm using Lee's algorithm for pathfinding.
- Enhanced `gen_pcb.py` to integrate routing capabilities, including segment generation for both front and back copper layers.
- Added functions to manage pad placement and via creation adjacent to pads.
- Updated the PCB generation process to include routing results in the final output.
- Improved error handling and logging for unconnected pads during routing.
Routing:
- added copper zone on In2.Cu, net +3V0
- removed copper zone on B.Cu, net GND
Changed lines of the file:
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@@
 	)
 	(zone
-		(net 8)
-		(net_name "GND")
-		(layer "B.Cu")
-		(name "GND B.Cu")
+		(net 1)
+		(net_name "+3V0")
+		(layer "In2.Cu")
+		(name "+3V0 In2.Cu")
 		(hatch edge 0.5)
 		(connect_pads (clearance 0.2))
